Commit message: sliding fixes

File: src/robot_description/urdf/common_properties.xacro (robot description, xacro)
@@ -58,5 +58,5 @@
         <inertia ixx="0.000166667" iyy = "0.000166667" izz="0.000166667" />
     </xacro:macro>
-   <xacro:macro name="wheel_link" params="prefix">
+    <xacro:macro name="wheel_link" params="prefix">
         <link name="${prefix}_wheel_link">
             <visual>
@@ -73,10 +73,9 @@
                 <origin xyz="0 0 0" rpy="${pi / 2.0} 0 0" />
             </collision>
-            <fdir1 value="1 0 0"/>
-            <xacro:sphere_inertia m="0.01" r="${wheel_radius}"
+            <xacro:sphere_inertia m="1.0" r="${wheel_radius}"
                                     o_xyz="0 0 0" o_rpy="${pi / 2.0} 0 0" />
         </link>
     </xacro:macro>
-    <xacro:macro name = "wheel_joint" params = "child_prefix xyz xyz_axis rpy joint_type:=fixed">
+    <xacro:macro name="wheel_joint" params="child_prefix xyz xyz_axis rpy joint_type:=fixed">
         <joint name="base_${child_prefix}_wheel_joint" type="${joint_type}">
             <parent link="base_link" />
@@ -84,4 +83,5 @@
             <origin xyz="${xyz}" rpy="${rpy}" />
             <axis xyz="${xyz_axis}" />
+            <dynamics damping="0.2" friction="0.2"/>
         </joint>
     </xacro:macro>

File: src/robot_description/urdf/gazebo_properties.xacro (robot description, xacro)
@@ -63,7 +63,7 @@
             <joint_name>al_profile_connector_joint</joint_name>
             <topic>/slider_z_cmd</topic>
-            <p_gain>10000</p_gain>
-            <i_gain>100</i_gain>
-            <d_gain>1000</d_gain>
+            <p_gain>100.0</p_gain>
+            <i_gain>0.1</i_gain>
+            <d_gain>5.0</d_gain>
         </plugin>
     </gazebo>
@@ -73,15 +73,16 @@
             <joint_name>al_profile2_joint</joint_name>
             <topic>/slider_x_cmd</topic>
-            <p_gain>10000</p_gain>
-            <i_gain>100</i_gain>
-            <d_gain>1000</d_gain>
+            <p_gain>100.0</p_gain>
+            <i_gain>0.1</i_gain>
+            <d_gain>5.0</d_gain>
         </plugin>
     </gazebo>
     <!-- ============================================================ -->
-    <!-- Wheel friction                                                -->
+    <!-- Wheel friction                                               -->
     <!-- ============================================================ -->
     <gazebo reference="left_back_wheel_link">
         <mu1>1.0</mu1>
         <mu2>1.0</mu2>
+        <fdir1>1 0 0</fdir1>
         <kp>500000.0</kp>
         <kd>10.0</kd>
@@ -91,16 +92,20 @@
         <mu1>1.0</mu1>
         <mu2>1.0</mu2>
+        <fdir1>1 0 0</fdir1>
         <kp>500000.0</kp>
         <kd>10.0</kd>
         <minDepth>0.001</minDepth>
     </gazebo>
-    <!-- Low friction caster for smooth turning -->
+    <gazebo reference="caster_wheel_joint">
+        <preserveFixedJoint>true</preserveFixedJoint>
+    </gazebo>
     <gazebo reference="caster_wheel">
-        <mu1>0.001</mu1>
-        <mu2>0.001</mu2>
-        <kp>500000.0</kp>
-        <kd>10.0</kd>
+        <mu1>0.0</mu1>
+        <mu2>0.0</mu2>
+        <kp>1000000.0</kp>
+        <kd>100.0</kd>
+        <minDepth>0.001</minDepth>
+        <maxVel>1.0</maxVel>
     </gazebo>
-    <!-- Base link visual colour in Gazebo -->
     <gazebo reference="base_link">
         <material>

File: src/robot_description/urdf/mobile_base.xacro (robot description, xacro)
@@ -109,10 +109,10 @@
         <visual>
             <geometry>
-                <sphere radius="${wheel_radius/2.0 - 0.025}"/>
+                <sphere radius="${wheel_radius/2.0 - 0.026}"/>
             </geometry>
         </visual>
         <collision>
             <geometry>
-                <sphere radius="${wheel_radius/2.0 - 0.025}"/>
+                <sphere radius="${wheel_radius/2.0 - 0.026}"/>
             </geometry>
         </collision>

Commit message: replaced sliders with pitch/yaw cleaning head

File: src/robot_description/urdf/common_properties.xacro (robot description, xacro)
@@ -4,7 +4,7 @@
         <color rgba="0 0.6 0 1" />
     </material>
-  <material name="silver">
-    <color rgba="0.8 0.8 0.8 1.0"/>
-  </material>
+    <material name="silver">
+        <color rgba="0.8 0.8 0.8 1.0"/>
+    </material>
     <material name="gray">
         <color rgba="0.7 0.7 0.7 1" />
@@ -12,4 +12,10 @@
     <material name = "black">
         <color rgba="0 0 0 1"/>
+    </material>
+    <material name = "blue">
+        <color rgba="0 0 1 1.0"/>
+    </material>
+    <material name = "water">
+        <color rgba="0 0 1 0.5"/>
     </material>
     <xacro:macro name="box_inertia" params="m x y z o_xyz o_rpy">

File: src/robot_description/urdf/gazebo_properties.xacro (robot description, xacro)
@@ -27,6 +27,6 @@
             <joint_name>base_left_back_wheel_joint</joint_name>
             <joint_name>base_right_back_wheel_joint</joint_name>
-            <joint_name>al_profile_connector_joint</joint_name>
-            <joint_name>al_profile2_joint</joint_name>
+            <joint_name>cleaning_head_pitch_joint</joint_name>
+            <joint_name>cleaning_head_yaw_joint</joint_name>
             <topic>/joint_states</topic>
             <update_rate>10</update_rate>
@@ -61,6 +61,6 @@
         <plugin filename="gz-sim-joint-position-controller-system"
                 name="gz::sim::systems::JointPositionController">
-            <joint_name>al_profile_connector_joint</joint_name>
-            <topic>/slider_z_cmd</topic>
+            <joint_name>cleaning_head_pitch_joint</joint_name>
+            <topic>/cleaning_head_pitch_target_cmd</topic>
             <p_gain>100.0</p_gain>
             <i_gain>0.1</i_gain>
@@ -71,6 +71,6 @@
         <plugin filename="gz-sim-joint-position-controller-system"
                 name="gz::sim::systems::JointPositionController">
-            <joint_name>al_profile2_joint</joint_name>
-            <topic>/slider_x_cmd</topic>
+            <joint_name>cleaning_head_yaw_joint</joint_name>
+            <topic>/cleaning_head_yaw_target_cmd</topic>
             <p_gain>100.0</p_gain>
             <i_gain>0.1</i_gain>

File: src/robot_description/urdf/mobile_base.xacro (robot description, xacro)
@@ -9,7 +9,9 @@
     <xacro:property name="al_profile_depth" value="0.04" />
     <xacro:property name="al_profile_height" value="1.45" />
-    <xacro:property name="al_profile2_length" value="1.0" />
+    <xacro:property name="al_profile2_length" value="0.6" />
     <xacro:property name="al_profile2_width" value="0.04" />
     <xacro:property name="al_profile2_depth" value="0.08" />
+    <xacro:property name="cleaning_head_pitch_height" value="0.05" />
+    <xacro:property name="cleaning_head_yaw_height" value="0.05" />
     <link name="base_footprint" />
     <link name="base_link">
@@ -46,20 +48,4 @@
         <xacro:box_inertia m="5.0" x="${al_profile_width}" y="${al_profile_depth}" z="${al_profile_height}" o_xyz="0 0 ${al_profile_height/2.0}" o_rpy="0 0 0" />
     </link>
-    <link name="al_profile_connector_link">
-        <visual>
-            <geometry>
-                <box size="0.1 0.1 0.1" />
-            </geometry>
-            <origin xyz="0 0 ${al_profile_height/2.0}" rpy="0 0 0" />
-            <material name="silver" />
-        </visual>
-        <collision>
-            <geometry>
-                <box size="0.1 0.1 0.1" />
-            </geometry>
-            <origin xyz="0 0 ${al_profile_height/2.0}" rpy="0 0 0" />
-        </collision>
-        <xacro:box_inertia m="0.1" x="0.1" y="0.1" z="0.1" o_xyz="0 0 ${al_profile_height/2.0}" o_rpy="0 0 0" />
-    </link>
     <link name="al_profile2_link">
         <visual>
@@ -67,5 +53,5 @@
                 <box size="${al_profile2_length} ${al_profile2_width} ${al_profile2_depth}" />
             </geometry>
-            <origin xyz="0 0 0" rpy="0 0 0" />
+            <origin xyz="0 0 0" rpy="0 0 1.5708" />
             <material name="silver" />
         </visual>
@@ -74,7 +60,40 @@
                 <box size="${al_profile2_length} ${al_profile2_width} ${al_profile2_depth}" />
             </geometry>
+            <origin xyz="0 0 0" rpy="0 0 1.5708" />
+        </collision>
+        <xacro:box_inertia m="3.0" x="${al_profile2_length}" y="${al_profile2_width}" z="${al_profile2_depth}" o_xyz="0 0 0" o_rpy="0 0 1.5708" />
+    </link>
+    <link name="cleaning_head_pitch_link">
+        <visual>
+            <geometry>
+                <box size="${cleaning_head_pitch_height} ${cleaning_head_pitch_height} ${cleaning_head_pitch_height}" />
+            </geometry>
+            <material name="black" />
             <origin xyz="0 0 0" rpy="0 0 0" />
-        </collision>
-        <xacro:box_inertia m="0.1" x="${al_profile2_length}" y="${al_profile2_width}" z="${al_profile2_depth}" o_xyz="0 0 0" o_rpy="0 0 1.5708" />
+        </visual>
+        <xacro:box_inertia m="0.1" x="0.030" y="0.040" z="0.030"
+                           o_xyz="0 0 0" o_rpy="0 0 0" />
+    </link>
+    <link name="cleaning_head_yaw_link">
+         <visual>
+            <geometry>
+                <cylinder radius="${cleaning_head_pitch_height/2.0}" length="${cleaning_head_yaw_height}"/>
+            </geometry>
+            <material name="green" />
+            <origin xyz="0 0 0" rpy="0 0 0" />
+        </visual>
+        <xacro:box_inertia m="0.1" x="0.030" y="0.040" z="0.030"
+                           o_xyz="0 0 0" o_rpy="0 0 0" />
+    </link>
+    <link name="cleaning_head_nozzle_link">
+         <visual>
+            <geometry>
+                <cylinder radius="${cleaning_head_yaw_height/4.0}" length="${cleaning_head_yaw_height*2.0}"/>
+            </geometry>
+            <material name="blue" />
+            <origin xyz="0 0 0" rpy="0 0 0" />
+        </visual>
+        <xacro:box_inertia m="0.1" x="0.030" y="0.040" z="0.030"
+                           o_xyz="0 0 0" o_rpy="0 0 0" />
     </link>
     <link name="camera_link">
@@ -104,15 +123,13 @@
     <xacro:wheel_link prefix="right_back" />
     <xacro:wheel_link prefix="left_back" />
-    <!-- In sim mode, wheels must be 'continuous' for Gazebo diff_drive plugin -->
-    <xacro:property name="wheel_jt" value="${'continuous' if sim_mode else 'fixed'}" />
     <link name="caster_wheel">
         <visual>
             <geometry>
-                <sphere radius="${wheel_radius/2.0 - 0.026}"/>
+                <sphere radius="${wheel_radius/2.0 - 0.025}"/>
             </geometry>
         </visual>
         <collision>
             <geometry>
-                <sphere radius="${wheel_radius/2.0 - 0.026}"/>
+                <sphere radius="${wheel_radius/2.0 - 0.025}"/>
             </geometry>
         </collision>
@@ -124,4 +141,5 @@
         <origin xyz="0 0 ${-wheel_radius}" rpy="0 0 0" />
     </joint>
+    <xacro:property name="wheel_jt" value="${'continuous' if sim_mode else 'fixed'}" />
     <xacro:wheel_joint child_prefix = "left_back" xyz = "${(-base_length / 2.0)+0.123} ${(base_width + wheel_length) / 2.0 } 0.025" xyz_axis = "0 1 0" rpy = "0 0 0" joint_type="${wheel_jt}"/>
     <xacro:wheel_joint child_prefix = "right_back" xyz = "${(-base_length / 2.0)+0.123} ${-(base_width + wheel_length) / 2.0 } 0.025" xyz_axis = "0 1 0" rpy = "0 0 0" joint_type="${wheel_jt}"/>
@@ -136,20 +154,32 @@
         <origin xyz="0 0 ${base_height}" rpy="0 0 0" />
     </joint>
-    <joint name="al_profile_connector_joint" type="prismatic">
+    <joint name="al_profile2_joint" type="fixed">
         <parent link="al_profile_link" />
-        <child link="al_profile_connector_link" />
-        <origin xyz="0 0 ${base_height}" rpy="0 0 0" />
-        <axis xyz="0 0 1" /> <limit lower="${-al_profile_height/2.0}" upper="${al_profile_height/2.0 - base_height - 0.1}" effort="100.0" velocity="0.5" />
+        <child link="al_profile2_link" />
+        <origin xyz="${al_profile_width} 0 ${al_profile_height/2.0}" rpy="0 0 0" />
     </joint>
-    <joint name="al_profile2_joint" type="prismatic">
-        <parent link="al_profile_connector_link" />
-        <child link="al_profile2_link" />
-        <origin xyz="0 0 ${al_profile_height/2.0}" rpy="0 0 0" />
-        <axis xyz="1 0 0" /> <limit lower="${-al_profile2_length/2.0}" upper="${al_profile2_length/2.0}" effort="100.0" velocity="0.5" />
+    <joint name="cleaning_head_pitch_joint" type="revolute">
+        <parent link="al_profile2_link" />
+        <child link="cleaning_head_pitch_link" />
+        <origin xyz="0 ${-al_profile2_length/2.0 + cleaning_head_pitch_height/2.0} ${al_profile2_width + cleaning_head_pitch_height/2.0}" rpy="0 0 0" />
+        <axis xyz="1 0 0" />
+        <limit lower="${-pi/2.0}" upper="${pi/2.0}" effort="10.0" velocity="1.0" />
+    </joint>
+    <joint name="cleaning_head_yaw_joint" type="revolute">
+        <parent link="cleaning_head_pitch_link" />
+        <child link="cleaning_head_yaw_link" />
+        <origin xyz="0 0 ${cleaning_head_pitch_height}" rpy="0 0 0" />
+        <axis xyz="0 0 1" />
+        <limit lower="${-pi/2.0}" upper="${pi/2.0}" effort="10.0" velocity="1.0" />
+    </joint>
+    <joint name="cleaning_head_nozzle_joint" type="fixed">
+        <parent link="cleaning_head_yaw_link" />
+        <child link="cleaning_head_nozzle_link" />
+        <origin xyz="0 -${cleaning_head_yaw_height - 0.01} 0" rpy="${pi/2.0} 0 0" />
     </joint>
     <joint name="camera_joint" type="fixed">
-        <parent link="al_profile_link" />
+        <parent link="al_profile2_link" />
         <child link="camera_link" />
-        <origin xyz="0 0 ${al_profile_height+0.015}" rpy="0 0.26179 -1.5708" />
+        <origin xyz="0 ${-al_profile2_length/2.0} 0" rpy="0 0 -1.5708" />
     </joint>
 </robot>
