Commit message: xz sliders!

File: src/robot_description/urdf/gazebo_properties.xacro (robot description, xacro)
@@ -1,19 +1,4 @@
 <?xml version="1.0"?>
-<!--
-  gazebo_properties.xacro — Gazebo Harmonic simulation plugins.
-  Conditionally included by robot.xacro when use_sim:=true.
-  Provides physics simulation for the differential-drive robot:
-  Plugins:
-    - DiffDrive         — Subscribes to /cmd_vel, publishes /odom + TF
-    - JointStatePublisher — Publishes /joint_states for wheel joints
-    - 3D GPU LiDAR      — Simulates Unitree L1 (360° × 18-line, 25 m range)
-    - IMU sensor         — 200 Hz accelerometer + gyroscope on base_link
-  Topic names use absolute paths so the ros_gz_bridge can map them
-  directly to ROS 2 topics without model-name scoping.
--->
 <robot xmlns:xacro="http://www.ros.org/wiki/xacro">
-    <!-- ============================================================ -->
-    <!-- Differential Drive Controller                                 -->
-    <!-- ============================================================ -->
     <gazebo>
         <plugin filename="gz-sim-diff-drive-system"
@@ -37,7 +22,4 @@
         </plugin>
     </gazebo>
-    <!-- ============================================================ -->
-    <!-- Joint State Publisher (wheel rotations)                       -->
-    <!-- ============================================================ -->
     <gazebo>
         <plugin filename="gz-sim-joint-state-publisher-system"
@@ -45,72 +27,10 @@
             <joint_name>base_left_back_wheel_joint</joint_name>
             <joint_name>base_right_back_wheel_joint</joint_name>
+            <joint_name>al_profile_connector_joint</joint_name>
+            <joint_name>al_profile2_joint</joint_name>
             <topic>/joint_states</topic>
             <update_rate>10</update_rate>
         </plugin>
     </gazebo>
-    <!-- ============================================================ -->
-    <!-- 3D LiDAR sensor (simulates Unitree L1)                       -->
-    <!-- 360° horizontal, ~18 vertical lines, 25 m range, 10 Hz       -->
-    <!-- ============================================================ -->
-    <gazebo reference="lidar_link">
-        <sensor name="lidar" type="gpu_lidar">
-            <topic>/scan/points</topic>
-            <update_rate>10</update_rate>
-            <always_on>true</always_on>
-            <visualize>true</visualize>
-            <lidar>
-                <scan>
-                    <horizontal>
-                        <samples>360</samples>
-                        <resolution>1</resolution>
-                        <min_angle>-3.14159</min_angle>
-                        <max_angle>3.14159</max_angle>
-                    </horizontal>
-                    <vertical>
-                        <samples>18</samples>
-                        <resolution>1</resolution>
-                        <min_angle>-0.2618</min_angle>
-                        <max_angle>0.7854</max_angle>
-                    </vertical>
-                </scan>
-                <range>
-                    <min>0.1</min>
-                    <max>25.0</max>
-                    <resolution>0.01</resolution>
-                </range>
-                <noise>
-                    <type>gaussian</type>
-                    <mean>0</mean>
-                    <stddev>0.005</stddev>
-                </noise>
-            </lidar>
-        </sensor>
-    </gazebo>
-    <!-- ============================================================ -->
-    <!-- IMU sensor on base_link (200 Hz)                              -->
-    <!-- ============================================================ -->
-    <gazebo reference="base_link">
-        <sensor name="imu" type="imu">
-            <topic>/imu/data</topic>
-            <update_rate>200</update_rate>
-            <always_on>true</always_on>
-            <imu>
-                <angular_velocity>
-                    <x><noise type="gaussian"><mean>0</mean><stddev>0.0002</stddev></noise></x>
-                    <y><noise type="gaussian"><mean>0</mean><stddev>0.0002</stddev></noise></y>
-                    <z><noise type="gaussian"><mean>0</mean><stddev>0.0002</stddev></noise></z>
-                </angular_velocity>
-                <linear_acceleration>
-                    <x><noise type="gaussian"><mean>0</mean><stddev>0.017</stddev></noise></x>
-                    <y><noise type="gaussian"><mean>0</mean><stddev>0.017</stddev></noise></y>
-                    <z><noise type="gaussian"><mean>0</mean><stddev>0.017</stddev></noise></z>
-                </linear_acceleration>
-            </imu>
-        </sensor>
-    </gazebo>
-    <!-- ============================================================ -->
-    <!-- RGB Camera sensor (top of al_profile_link, faces +x/forward) -->
-    <!-- 640×480 @ 30 Hz, 80° horizontal FOV                          -->
-    <!-- ============================================================ -->
     <gazebo reference="camera_link">
         <sensor name="camera" type="camera">
@@ -137,4 +57,24 @@
             </camera>
         </sensor>
+    </gazebo>
+    <gazebo>
+        <plugin filename="gz-sim-joint-position-controller-system"
+                name="gz::sim::systems::JointPositionController">
+            <joint_name>al_profile_connector_joint</joint_name>
+            <topic>/slider_z_cmd</topic>
+            <p_gain>10000</p_gain>
+            <i_gain>100</i_gain>
+            <d_gain>1000</d_gain>
+        </plugin>
+    </gazebo>
+    <gazebo>
+        <plugin filename="gz-sim-joint-position-controller-system"
+                name="gz::sim::systems::JointPositionController">
+            <joint_name>al_profile2_joint</joint_name>
+            <topic>/slider_x_cmd</topic>
+            <p_gain>10000</p_gain>
+            <i_gain>100</i_gain>
+            <d_gain>1000</d_gain>
+        </plugin>
     </gazebo>
     <!-- ============================================================ -->

File: src/robot_description/urdf/mobile_base.xacro (robot description, xacro)
@@ -9,5 +9,5 @@
     <xacro:property name="al_profile_depth" value="0.04" />
     <xacro:property name="al_profile_height" value="1.45" />
-    <xacro:property name="al_profile2_length" value="0.6" />
+    <xacro:property name="al_profile2_length" value="1.0" />
     <xacro:property name="al_profile2_width" value="0.04" />
     <xacro:property name="al_profile2_depth" value="0.08" />
@@ -46,4 +46,20 @@
         <xacro:box_inertia m="5.0" x="${al_profile_width}" y="${al_profile_depth}" z="${al_profile_height}" o_xyz="0 0 ${al_profile_height/2.0}" o_rpy="0 0 0" />
     </link>
+    <link name="al_profile_connector_link">
+        <visual>
+            <geometry>
+                <box size="0.1 0.1 0.1" />
+            </geometry>
+            <origin xyz="0 0 ${al_profile_height/2.0}" rpy="0 0 0" />
+            <material name="silver" />
+        </visual>
+        <collision>
+            <geometry>
+                <box size="0.1 0.1 0.1" />
+            </geometry>
+            <origin xyz="0 0 ${al_profile_height/2.0}" rpy="0 0 0" />
+        </collision>
+        <xacro:box_inertia m="0.1" x="0.1" y="0.1" z="0.1" o_xyz="0 0 ${al_profile_height/2.0}" o_rpy="0 0 0" />
+    </link>
     <link name="al_profile2_link">
         <visual>
@@ -51,5 +67,5 @@
                 <box size="${al_profile2_length} ${al_profile2_width} ${al_profile2_depth}" />
             </geometry>
-            <origin xyz="0 0 0" rpy="0 0 1.5708" />
+            <origin xyz="0 0 0" rpy="0 0 0" />
             <material name="silver" />
         </visual>
@@ -58,7 +74,7 @@
                 <box size="${al_profile2_length} ${al_profile2_width} ${al_profile2_depth}" />
             </geometry>
-            <origin xyz="0 0 0" rpy="0 0 1.5708" />
+            <origin xyz="0 0 0" rpy="0 0 0" />
         </collision>
-        <xacro:box_inertia m="3.0" x="${al_profile2_length}" y="${al_profile2_width}" z="${al_profile2_depth}" o_xyz="0 0 0" o_rpy="0 0 1.5708" />
+        <xacro:box_inertia m="0.1" x="${al_profile2_length}" y="${al_profile2_width}" z="${al_profile2_depth}" o_xyz="0 0 0" o_rpy="0 0 1.5708" />
     </link>
     <link name="camera_link">
@@ -86,39 +102,4 @@
                            o_xyz="0 0 0" o_rpy="0 0 0" />
     </link>
-    <link name = "lidar_link">
-        <visual>
-            <geometry>
-                <cylinder radius="0.0375" length="0.065" />
-            </geometry>
-            <origin xyz="0 0 0" rpy="0 0 0" />
-            <material name="black" />
-        </visual>
-        <collision>
-            <geometry>
-                <cylinder radius="0.0375" length="0.065" />
-            </geometry>
-            <origin xyz="0 0 0" rpy="0 0 0" />
-        </collision>
-        <xacro:box_inertia m="0.1" x="0.075" y="0.075" z="0.065"
-                           o_xyz="0 0 0" o_rpy="0 0 0" />
-    </link>
-    <!--
-    <link name = "unilidar_imu">
-        <visual>
-            <geometry>
-                <box size="0.025 0.025 0.025" />
-            </geometry>
-            <origin xyz="0 0 0" rpy="0 0 0" />
-            <material name="silver" />
-        </visual>
-        <collision>
-            <geometry>
-                <box size="0.025 0.025 0.025" />
-            </geometry>
-            <origin xyz="0 0 0" rpy="0 0 0" />
-        </collision>
-        <xacro:box_inertia m="0.05" x="0.025" y="0.025" z="0.025"
-                           o_xyz="0 0 0" o_rpy="0 0 0" />
-    </link> -->
     <xacro:wheel_link prefix="right_back" />
     <xacro:wheel_link prefix="left_back" />
@@ -133,5 +114,5 @@
         <collision>
             <geometry>
-                <sphere radius="${wheel_radius/2.0 - 0.01}"/>
+                <sphere radius="${wheel_radius/2.0 - 0.025}"/>
             </geometry>
         </collision>
@@ -150,20 +131,4 @@
         <origin xyz="${base_length/2 - 0.09} 0 ${-wheel_radius/2}"/>
     </joint>
-    <!-- Sim: base_link is root, lidar is a child (Gazebo diff_drive publishes odom→base_link) -->
-    <xacro:if value="${sim_mode}">
-        <joint name="lidar_base_link_joint" type="fixed">
-            <parent link="base_link"/>
-            <child link="lidar_link"/>
-            <origin xyz="${al_profile_width} 0 ${((al_profile_height+base_height+wheel_radius/2)-0.14)}" rpy="3.1416 0 -0.3926"/>
-        </joint>
-    </xacro:if>
-    <!-- Real hardware: lidar_link is root (Point-LIO publishes odom→lidar_link) -->
-    <xacro:unless value="${sim_mode}">
-        <joint name="lidar_base_link_joint" type="fixed">
-            <parent link="lidar_link"/>
-            <child link="base_link"/>
-            <origin xyz="${al_profile_width} ${-(0.065/2)} ${((al_profile_height+base_height+wheel_radius/2)-0.14)}" rpy="3.1416 0 -0.3926"/>
-        </joint>
-    </xacro:unless>
     <joint name="al_profile_joint" type="fixed">
         <parent link="base_link" />
@@ -171,8 +136,15 @@
         <origin xyz="0 0 ${base_height}" rpy="0 0 0" />
     </joint>
-    <joint name="al_profile2_joint" type="fixed">
+    <joint name="al_profile_connector_joint" type="prismatic">
         <parent link="al_profile_link" />
+        <child link="al_profile_connector_link" />
+        <origin xyz="0 0 ${base_height}" rpy="0 0 0" />
+        <axis xyz="0 0 1" /> <limit lower="${-al_profile_height/2.0}" upper="${al_profile_height/2.0 - base_height - 0.1}" effort="100.0" velocity="0.5" />
+    </joint>
+    <joint name="al_profile2_joint" type="prismatic">
+        <parent link="al_profile_connector_link" />
         <child link="al_profile2_link" />
-        <origin xyz="${al_profile_width} 0 ${al_profile_height/2.0}" rpy="0 0 0" />
+        <origin xyz="0 0 ${al_profile_height/2.0}" rpy="0 0 0" />
+        <axis xyz="1 0 0" /> <limit lower="${-al_profile2_length/2.0}" upper="${al_profile2_length/2.0}" effort="100.0" velocity="0.5" />
     </joint>
     <joint name="camera_joint" type="fixed">
@@ -181,8 +153,3 @@
         <origin xyz="0 0 ${al_profile_height+0.015}" rpy="0 0.26179 -1.5708" />
     </joint>
-    <!-- <joint name="imu_lidar_joint" type="fixed">
-        <parent link="unilidar_imu"/>
-        <child link="lidar_link"/>
-        <origin xyz="0.007698 0.014655 -0.00667"/>
-    </joint> -->
 </robot>

Commit message: Cleaning head movement + broken UI :(

File: src/robot_description/urdf/gazebo_properties.xacro (robot description, xacro)
@@ -40,5 +40,5 @@
             <visualize>true</visualize>
             <camera>
-                <horizontal_fov>1.3962634</horizontal_fov>
+                <horizontal_fov>${pi/2.0}</horizontal_fov>
                 <image>
                     <width>640</width>
@@ -58,4 +58,34 @@
         </sensor>
     </gazebo>
+    <gazebo reference="cleaning_head_nozzle_link">
+      <sensor name="water_stream_sensor" type="gpu_lidar">
+        <gz_frame_id>water_nozzle_link</gz_frame_id>
+        <topic>/water_hit_scan</topic>
+        <update_rate>30</update_rate>
+        <always_on>1</always_on>
+        <visualize>true</visualize>
+        <ray>
+          <scan>
+            <horizontal>
+              <samples>1</samples>
+              <resolution>1</resolution>
+              <min_angle>0</min_angle>
+              <max_angle>0</max_angle>
+            </horizontal>
+            <vertical>
+              <samples>1</samples>
+              <resolution>1</resolution>
+              <min_angle>${pi/2.0}</min_angle>
+              <max_angle>${pi/2.0}</max_angle>
+            </vertical>
+          </scan>
+          <range>
+            <min>0.1</min>
+            <max>5.0</max>
+            <resolution>0.01</resolution>
+          </range>
+        </ray>
+      </sensor>
+    </gazebo>
     <gazebo>
         <plugin filename="gz-sim-joint-position-controller-system"
@@ -63,7 +93,9 @@
             <joint_name>cleaning_head_pitch_joint</joint_name>
             <topic>/cleaning_head_pitch_target_cmd</topic>
-            <p_gain>100.0</p_gain>
-            <i_gain>0.1</i_gain>
-            <d_gain>5.0</d_gain>
+            <p_gain>1000.0</p_gain>
+            <i_gain>5.0</i_gain>
+            <d_gain>2.0</d_gain>
+            <i_max>15.0</i_max>
+            <i_min>-15.0</i_min>
         </plugin>
     </gazebo>
@@ -73,7 +105,9 @@
             <joint_name>cleaning_head_yaw_joint</joint_name>
             <topic>/cleaning_head_yaw_target_cmd</topic>
-            <p_gain>100.0</p_gain>
-            <i_gain>0.1</i_gain>
-            <d_gain>5.0</d_gain>
+            <p_gain>1000.0</p_gain>
+            <i_gain>2.0</i_gain>
+            <d_gain>1.0</d_gain>
+            <i_max>5.0</i_max>
+            <i_min>-5.0</i_min>
         </plugin>
     </gazebo>
@@ -114,3 +148,8 @@
         </material>
     </gazebo>
+    <gazebo>
+        <frame name="lidar_frame" attached_to='cleaning_head_nozzle_link'>
+            <pose>0.0 0.0 0.0 0 0 0</pose>
+        </frame>
+    </gazebo>
 </robot>

File: src/robot_description/urdf/mobile_base.xacro (robot description, xacro)
@@ -97,4 +97,13 @@
                            o_xyz="0 0 0" o_rpy="0 0 0" />
     </link>
+    <link name="cleaning_head_water_link">
+         <visual>
+            <geometry>
+                <cylinder radius="${cleaning_head_yaw_height/6.0}" length="${5}"/>
+            </geometry>
+            <material name="water" />
+            <origin xyz="0 0 0" rpy="0 0 0" />
+        </visual>
+    </link>
     <link name="camera_link">
         <visual>
@@ -178,4 +187,9 @@
         <origin xyz="0 -${cleaning_head_yaw_height - 0.01} 0" rpy="${pi/2.0} 0 0" />
     </joint>
+    <joint name="cleaning_head_water_joint" type="fixed">
+        <parent link="cleaning_head_nozzle_link" />
+        <child link="cleaning_head_water_link" />
+        <origin xyz="0 0 2.5" rpy="0 0 0" />
+    </joint>
     <joint name="camera_joint" type="fixed">
         <parent link="al_profile2_link" />
